File: base/noroshi_LoRa_RAK.brd (EAGLE design)
At the start: 40.5 x 35 mm, 20 parts

Commit message: Update noroshi.
Parts:
- removed LED2, LED3: (no value), FaBo-LED:0603
- removed R7, R8: 470, FaBo-Resistors:0603-NARROW
- removed R9: 10k, FaBo-Resistors:0603-NARROW
- added C2: 4.7uF, FaBo-Capacitor:0603-NARROW
- added C7, C8: 0.1uF, FaBo-Capacitor:0603-NARROW
- added JP1: (no value), adafruit:1X03
- added L1: (no value), FaBo-Coil:0603
- added UF1: (no value), FaBo-Connetor:HIROSE-UF.L
- U$2: value ES920LR -> RAK811; device FaBo-LoRa:ES920LR -> FaBo-LoRa:RAK811
- moved U$3 32.4 mm to (3.55, 12.2)
- moved C1 20.0 mm to (9.20, 33.1), turned to 90 degrees
- moved C6 14.8 mm to (12.0, 15.2)
- moved U$8 7.01 mm to (36.5, 15.1), turned to 270 degrees
- moved U$2 3.77 mm to (23.2, 26.2), turned to 180 degrees
- moved RESET1 1.33 mm to (2.34, 26.6), turned to 90 degrees
Connections:
- removed net N$4: LED3.CATHODE, U$2.19
- removed net N$5: LED2.CATHODE, U$2.20
- removed net N$6: LED2.ANODE, R7.1
- removed net N$7: LED3.ANODE, R8.1
- removed net N$8: R9.1, U$2.16
- new net BOOT: JP1.2, U$2.17
- new net N$2: C7.2, L1.2, U$2.33
- new net N$3: C8.2, L1.1, UF1.SIG
- net +3V3: no longer C1.2, R7.2, R8.2, R9.2, U$2.13, U$2.2
- net 3V3: now also C1.2, C2.2, JP1.1, U$2.11
- net ANALOG: now also U$2.23; no longer U$2.12
- net GND: now also C2.1, C7.1, C8.1, JP1.3, U$2.12, U$2.21, U$2.28, U$2.30, U$2.31, U$2.32, U$2.34, UF1.GND@1, UF1.GND@2; no longer U$2.26, U$2.GND
- net RX: now also U$2.7; no longer U$2.9
- net SCL: now also U$2.18; no longer U$2.10
- net SDA: now also U$2.19; no longer U$2.11
- net SWD_CLK: now also U$2.13; no longer U$2.5
- net SWD_DIO: now also U$2.10; no longer U$2.6
- net TX: now also U$2.6; no longer U$2.8
Routing:
- net GND: track 130.9 -> 0.00 mm, vias 28 -> 20
- net 3V3: track 0.00 -> 54.4 mm
- net N$6: track 43.4 -> 0.00 mm
- net SWD_CLK: track 28.6 -> 68.6 mm, vias 2 -> 0
- net N$2: track 0.00 -> 36.0 mm, vias 0 -> 2
- net N$7: track 29.2 -> 0.00 mm, vias 2 -> 0
- net +3V3: track 100.2 -> 76.0 mm, vias 0 -> 1
- net RESETB: track 45.6 -> 65.8 mm
- net SCL: track 33.4 -> 13.8 mm
- net BOOT: track 0.00 -> 16.9 mm
- net RX: track 45.6 -> 30.6 mm
- net N$4: track 12.5 -> 0.00 mm
- net SDA: track 27.4 -> 16.5 mm, vias 1 -> 0
- net N$8: track 9.71 -> 0.00 mm
- net N$5: track 8.25 -> 0.00 mm
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Other:
- board text added: "#2"
- board text added: "Boot"
- board text removed: "#1"
