File: base/noroshi_LoRa_RAK.sch (EAGLE design)
At the start: 18 parts

Commit message: Update noroshi.
Parts:
- removed LED2, LED3: (no value), FaBo-LED:LED-0603
- removed R7, R8: 470, FaBo-Resistors:RESISTOR-0603-NARROW
- removed R9: 10k, FaBo-Resistors:RESISTOR-0603-NARROW
- added C2: 4.7uF, FaBo-Capacitor:CAPACITOR-0603_NARROW
- added C7, C8: 0.1uF, FaBo-Capacitor:CAPACITOR-0603_NARROW
- added JP1: (no value), adafruit:PINHD-1X3
- added L1: (no value), FaBo-Coil:COIL-0603
- added UF1: (no value), FaBo-Connetor:HIROSE-U.FL
- U$2: value ES920LR -> RAK811; device FaBo-LoRa:ES920LR -> FaBo-LoRa:RAK811
Connections:
- removed net N$4: LED3.CATHODE, U$2.PTE16/PCS
- removed net N$5: LED2.CATHODE, U$2.PTE17/SCK
- removed net N$6: LED2.ANODE, R7.1
- removed net N$7: LED3.ANODE, R8.1
- removed net N$8: R9.1, U$2.PTC1/SW_INT
- new net BOOT: JP1.2, U$2.BOOT0
- new net N$2: C7.2, L1.2, U$2.RF_OUT
- new net N$3: C8.2, L1.1, UF1.SIG
- net +3V3: no longer C1.2, R7.2, R8.2, R9.2, U$2.VCC, U$2.VCCRF
- net 3V3: now also C1.2, C2.2, JP1.1, U$2.VCC
- net ANALOG: now also U$2.PA0; no longer U$2.PTE30/DACO
- net GND: now also C2.1, C7.1, C8.1, JP1.3, U$2.GND@12, U$2.GND@21, U$2.GND@28, U$2.GND@30, U$2.GND@31, U$2.GND@32, U$2.GND@34, UF1.GND; no longer U$2.GND, U$2.GND@26
- net RESETB: now also U$2.RST; no longer U$2.RESETB
- net RX: now also U$2.UART1_RX; no longer U$2.PTA1/RX
- net SCL: now also U$2.PB8; no longer U$2.PTB0/SCL
- net SDA: now also U$2.PB9; no longer U$2.PTB1/SDA
- net SWD_CLK: now also U$2.PA14; no longer U$2.PTA0/SWD_CLK
- net SWD_DIO: now also U$2.PA13; no longer U$2.PTA3/SWD_DIO
- net TX: now also U$2.UART1_TX; no longer U$2.PTA2/TX
Other:
- moved on the sheet: C1
